File: plates/pcb-top/plate-top.kicad_pcb (KiCad board)
At the start: 2 copper layers, 152 x 91.6 mm, 22 parts, among them K1 SW_Push, K10 SW_Push, K11 SW_Push, K12 SW_Push, K13 SW_Push, K14 SW_Push, K15 SW_Push, K16 SW_Push, K17 SW_Push, K18 SW_Push, K19 SW_Push, K2 SW_Push, K20 SW_Push, K21 SW_Push, K3 SW_Push, K4 SW_Push, K5 SW_Push, K6 SW_Push, K7 SW_Push, K8 SW_Push, K9 SW_Push, SW30 Rotary_Encoder_Switch

Commit message: cirrus40, second manufactured version
Parts:
- removed K19, K20, K21: SW_Push, footprints:Switch_Hole_Dogbone
- added REF**: MountingHole_2.2mm_M2, MountingHole:MountingHole_2.2mm_M2, F.Cu at (172.1, 110.5)
- added REF**: MountingHole_2.2mm_M2, MountingHole:MountingHole_2.2mm_M2, F.Cu at (172.1, 96.5)
- added REF**: MountingHole_2.2mm_M2, MountingHole:MountingHole_2.2mm_M2, F.Cu at (158.0, 96.5)
- added REF**: MountingHole_2.2mm_M2, MountingHole:MountingHole_2.2mm_M2, F.Cu at (158.0, 110.5)
- added REF**: MountingHole_2.2mm_M2, MountingHole:MountingHole_2.2mm_M2, F.Cu at (78.5, 65.9)
- added REF**: MountingHole_2.2mm_M2, MountingHole:MountingHole_2.2mm_M2, F.Cu at (135.5, 64.2)
- added REF**: MountingHole_2.2mm_M2, MountingHole:MountingHole_2.2mm_M2, F.Cu at (129.2, 126.2)
- added REF**: MountingHole_2.2mm_M2, MountingHole:MountingHole_2.2mm_M2, F.Cu at (78.5, 104.2)
- added REF**: MountingHole_2.2mm_M2, MountingHole:MountingHole_2.2mm_M2, F.Cu at (169.9, 131.6)
- added REF**: MountingHole_2.2mm_M2, MountingHole:MountingHole_2.2mm_M2, F.Cu at (135.5, 102.2)
- moved K10 0.64 mm to (140.3, 121.9)
- renumbered K13 to K1, K18 to K10, K4 to K11, K5 to K12, K6 to K13, K17 to K14, K1 to K15, K2 to K16, K3 to K17, K16 to K18, K14 to K2, K15 to K3, K10 to K4, K11 to K5, K12 to K6
Other:
- board size 152 x 91.6 mm -> 133.2 x 91.6 mm
